File: BE6502 SBC/BE6502 SBC.kicad_pcb (KiCad board)
At the start: 2 copper layers, 99.1 x 99.1 mm, 61 parts, among them J1 Expansion, J2 CLOCK_SEL, J3 BARREL_JACK, J4 Control, M1 Mounting, M2 Mounting, M3 Mounting, M4 Mounting, SW1 RESET, SW2 MIDDLE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

Commit message: make some basic changes
Connections:
- net /R/~W renamed /R/~{W}
- net /~IRQ renamed /~{IRQ}
- net /~NMI renamed /~{NMI}
- net /~RDY renamed /~{RDY}
- net ~RAM renamed ~{RAM}
- net ~RESET renamed ~{RESET}
- net ~ROM renamed ~{ROM}
- net ~VIA renamed ~{VIA}
Other:
- net class Default removed
- net class VCC removed
- board text added: "6K Machine"
- board text added: "MK67"
- board text added: "github.com/thepanoc95"
- board text removed: "Build a 65c02 computer"
- board text removed: "for video series by Ben Eater"
- board text removed: "github.com/tebl"

Commit message: Add a bunch of stuff
Parts:
- added J5: RCA_VIDEO, Connector:RCA_Phono_THT, F.Cu at (148.0, 108.5)
- added J6: PS2_KEYBOARD, Connector:PS2-6P_MiniDIN_THT, F.Cu at (148.0, 122.0)
- added R22: 1k, Resistors_THT:R_Axial_DIN0207_L6.3mm_D2.5mm_P10.16mm_Horizontal, F.Cu at (124.0, 101.0)
- added R23: 2k, Resistors_THT:R_Axial_DIN0207_L6.3mm_D2.5mm_P10.16mm_Horizontal, F.Cu at (124.0, 104.0)
- added R24: 4.7k, Resistors_THT:R_Axial_DIN0207_L6.3mm_D2.5mm_P10.16mm_Horizontal, F.Cu at (124.0, 107.0)
- added R25: 10k, Resistors_THT:R_Axial_DIN0207_L6.3mm_D2.5mm_P10.16mm_Horizontal, F.Cu at (124.0, 110.0)
- added R26: 22k, Resistors_THT:R_Axial_DIN0207_L6.3mm_D2.5mm_P10.16mm_Horizontal, F.Cu at (124.0, 113.0)
- added R27: 47k, Resistors_THT:R_Axial_DIN0207_L6.3mm_D2.5mm_P10.16mm_Horizontal, F.Cu at (124.0, 116.0)
- added R28: 4.7k, Resistors_THT:R_Axial_DIN0207_L6.3mm_D2.5mm_P10.16mm_Horizontal, F.Cu at (124.0, 120.0)
- added R29: 4.7k, Resistors_THT:R_Axial_DIN0207_L6.3mm_D2.5mm_P10.16mm_Horizontal, F.Cu at (124.0, 124.0)
